File: boards/Reflex_V1/PicoFightingBoard.kicad_pcb (KiCad board)
At the start: 4 copper layers, 96.1 x 45.2 mm, 73 parts, among them J1 Conn_01x04_Male, J10 Conn_01x04_Male, J11 Conn_01x04_Male, J12 Conn_01x04_Male, J13 Conn_01x04_Male, J14 Conn_01x02, J15 USB_C_Receptacle, J16 USB_B, J17 SANWA, J18 SEIMITSU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

Commit message: Initial Commit
Connections:
- J16 pad 2: /USB_D+ -> /USB_D-
- J16 pad 3: /USB_D- -> /USB_D+
Routing:
- net /USB_D+: track 41.6 -> 42.8 mm
- net /USB_D-: track 38.9 -> 40.1 mm
- net GND: vias 176 -> 177
- added copper zone on In2.Cu, net GND
